Commit message: Big changes for Jim

File: description/urdf/robot_core.xacro (robot description, xacro)
@@ -40,13 +40,13 @@
                 <!-- mesh filename="package://stingray/description/meshes/Stingray.stl" scale="0.001 0.001 0.001"/-->
                 <!-- mesh filename="/home/ubuntu/stingray_ws/src/stingray/description/meshes/Stingray.stl" scale="0.001 0.001 0.001"/-->
-                <mesh filename="file://home/ubuntu/stingray_ws/src/stingray/description/meshes/Stingray.stl" scale="0.001 0.001 0.001"/>
+                <mesh filename="file://$(find stingray)/description/meshes/Stingray.stl" scale="0.001 0.001 0.001"/>
             </geometry>
             <material name="gray"/>
         </visual>
-        <visual name="-chassis_rviz_visual">
+        <visual name="chassis_rviz_visual">
              <origin xyz="0.0 0.0 0.0" rpy="0.0 0.0 0.0"/>
             <geometry>
                 <!-- box size="${chassis_length} ${chassis_width} ${chassis_height}"/ -->
-                <mesh filename="package://stingray/description/meshes/Stingray.stl" scale="0.001 0.001 0.001"/>
+                <mesh filename="file://$(find stingray)/description/meshes/Stingray.stl" scale="0.001 0.001 0.001"/>
                 <!-- mesh filename="/home/ubuntu/stingray_ws/src/stingray/description/meshes/Stingray.stl" scale="0.001 0.001 0.001"/-->
                 <!-- mesh filename="file://home/ubuntu/stingray_ws/src/stingray/description/meshes/Stingray.stl" scale="0.001 0.001 0.001"/-->
@@ -71,5 +71,5 @@
         <child link="left_wheel_link"/>
         <origin xyz="0.0 0.13 0.0" rpy="-${pi/2} 0.0 0.0"/>
-        <axis xyz="0.0 0.0 1.0"/>
+        <axis xyz="0 0 1"/>
     </joint>
     <link name="left_wheel_link">
@@ -100,5 +100,5 @@
         <child link="right_wheel_link"/>
         <origin xyz="0.0 -0.13 0.0" rpy="${pi/2} 0.0 0.0"/>
-        <axis xyz="0.0 0.0 -1.0"/>
+        <axis xyz="0 0 -1"/>
     </joint>
     <link name="right_wheel_link">

File: description/urdf/robot_gazebo.xacro (robot description, xacro)
@@ -1,66 +1,97 @@
 <?xml version="1.0"?>
-<robot xmlns:xacro="http://www.ros.org/wiki/xacro"  name="robot">
-    <gazebo>
-        <!--plugin name='diff_drive' filename='libgazebo_ros_diff_drive.so'-->
-        <plugin filename="libgz_ros2_control-system.so"  name="gz_ros2_control::GazeboSimROS2ControlPlugin">
-            <xacro:property name="pkgpath" value="$(find stingray)"/>
-            <parameters>${pkgpath}/config/my_controllers.yaml</parameters>
-            <!-- Wheel Information -->
+<robot xmlns:xacro="http://www.ros.org/wiki/xacro" name="robot">
+  <gazebo>
+    <!--plugin name='diff_drive' filename='libgazebo_ros_diff_drive.so'-->
+    <plugin filename="libgz_ros2_control-system.so" name="gz_ros2_control::GazeboSimROS2ControlPlugin">
+      <xacro:property name="pkgpath" value="$(find stingray)"/>
+      <parameters>$(find stingray)/config/my_controllers.yaml</parameters>
+    </plugin>
+    <!-- Wheel Information
             <left_joint>left_wheel_joint</left_joint>
-            <right_joint>right_wheel_joint</right_joint>
-            <wheel_separation>0.26</wheel_separation>
-            <wheel_diameter>0.124</wheel_diameter>
-            <!-- Limits -->
-            <max_wheel_torque>200</max_wheel_torque>
-            <max_wheel_acceleration>10.0</max_wheel_acceleration>
-            <!-- Output -->
-            <odometry_frame>odom</odometry_frame>
-            <robot_base_frame>base_footprint</robot_base_frame>
-            <publish_odom>true</publish_odom>
-            <publish_odom_tf>true</publish_odom_tf>
-            <publish_wheel_tf>true</publish_wheel_tf>
-        </plugin>
-    </gazebo>
-    <gazebo reference="chassis_link">
-            <material>Gazebo/Gray</material>
-            <!--mesh><uri>filename="package://stingray/description/meshes/Stingray.stl" scale="0.001 0.001 0.001"</uri></mesh-->
-    </gazebo>
-    <gazebo reference="left_wheel_link">
-        <material>Gazebo/Green</material>
-    </gazebo>
-    <gazebo reference="left_wheel_marker_visual">
-        <material>Gazebo/White</material>
-    </gazebo>
-    <gazebo reference="right_wheel_link">
-        <material>Gazebo/Red</material>
-    </gazebo>
-    <gazebo reference="right_wheel_marker_visual">
-        <material>Gazebo/White</material>
-    </gazebo>
-    <gazebo reference="caster_wheel_link">
-        <material>Gazebo/White</material>
-        <mu1 value="0.001"/>
-        <mu2 value="0.001"/>
-    </gazebo>
-    <!-- ROS2 Control Configuration -->
-    <ros2_control name="Stingray" type="system">
-        <hardware>
-            <plugin>gz_ros2_control/GazeboSimSystem</plugin>
-        </hardware>
-        <!-- Joints Controlled -->
-        <joint name="left_wheel_joint">
-            <command_interface name="velocity"/>
-            <state_interface name="velocity"/>
-        </joint>
-        <joint name="right_wheel_joint">
-            <command_interface name="velocity"/>
-            <state_interface name="velocity"/>
-        </joint>
-    </ros2_control>
-    <gazebo>
-        <plugin filename="libgz_ros2_control-system.so" name="gz_ros2_control::GazeboSimROS2ControlPlugin">
-            <parameters>$(find stingray)/config/my_controllers.yaml</parameters>
-            <parameters>$(find stingray)/config/gaz_ros2_ctl_use_sim.yaml</parameters>
-        </plugin>
-    </gazebo>
+  <right_joint>right_wheel_joint</right_joint>
+  <wheel_separation>0.26</wheel_separation>
+  <wheel_diameter>0.124</wheel_diameter>
+  <max_wheel_torque>200</max_wheel_torque>
+  <max_wheel_acceleration>10.0</max_wheel_acceleration>
+  <odometry_frame>odom</odometry_frame>
+  <robot_base_frame>base_footprint</robot_base_frame>
+  <publish_odom>true</publish_odom>
+  <publish_odom_tf>true</publish_odom_tf>
+  <publish_wheel_tf>true</publish_wheel_tf>
+</plugin> -->
+  </gazebo>
+  <gazebo reference="chassis_link">
+    <material>Gazebo/Gray</material>
+    <!--mesh><uri>filename="package://stingray/description/meshes/Stingray.stl" scale="0.001 0.001 0.001"</uri></mesh-->
+  </gazebo>
+  <gazebo reference="left_wheel_link">
+    <material>Gazebo/Green</material>
+  </gazebo>
+  <gazebo reference="left_wheel_marker_visual">
+    <material>Gazebo/White</material>
+  </gazebo>
+  <gazebo reference="right_wheel_link">
+    <material>Gazebo/Red</material>
+  </gazebo>
+  <gazebo reference="right_wheel_marker_visual">
+    <material>Gazebo/White</material>
+  </gazebo>
+  <gazebo reference="caster_wheel_link">
+    <material>Gazebo/White</material>
+    <mu1 value="0.001"/>
+    <mu2 value="0.001"/>
+  </gazebo>
+  <!-- ROS2 Control Configuration -->
+  <ros2_control name="GazeboSystem" type="system">
+    <hardware>
+      <plugin>gz_ros2_control/GazeboSimSystem</plugin>
+    </hardware>
+    <!-- Joints Controlled -->
+    <joint name="left_wheel_joint">>
+      <command_interface name="velocity"
+        <param name="min">-10</param>
+        <param name="max">10</param>
+      </command_interface>
+      <state_interface name="velocity" />
+      <state_interface name="position" />
+    </joint>
+    <joint name="right_wheel_joint">
+      <command_interface name="velocity">
+        <param name="min">-10</param>
+        <param name="max">10</param>
+      </command_interface>
+      <state_interface name="velocity" />
+      <state_interface name="position" />
+    </joint>
+  </ros2_control>
+  <gazebo>
+    <plugin filename="libgz_ros2_control-system.so" name="gz_ros2_control::GazeboSimROS2ControlPlugin">
+      <parameters>$(find stingray)/config/my_controllers.yaml</parameters>
+      <parameters>$(find stingray)/config/gaz_ros2_ctl_use_sim.yaml</parameters>
+    </plugin>
+  </gazebo>
+  <gazebo>
+    <plugin filename="gz-sim-diff-drive-system" name="gz::sim::systems::DiffDrive">
+      <left_joint>left_wheel_joint</left_joint>
+      <right_joint>right_wheel_joint</right_joint>
+      <wheel_separation>0.26</wheel_separation>
+      <wheel_radius>0.028</wheel_radius>
+      <!-- Limits -->
+      <!-- <max_wheel_torque>200</max_wheel_torque> -->
+      <max_linear_acceleration>1.0</max_linear_acceleration>
+      <!-- Input -->
+      <topic>cmd_vel</topic>
+      <!-- Output -->
+      <frame_id>odom</frame_id>
+      <child_frame_id>base_footprint</child_frame_id>
+      <odom_topic>odom</odom_topic>
+      <odom_publisher_frequency>50</odom_publisher_frequency>
+      <tf_topic>/tf</tf_topic>
+    </plugin>
+    <plugin filename="gz-sim-joint-state-publisher-system" name="gz::sim::systems::JointStatePublisher">
+      <topic>joint_states</topic>
+      <joint_name>left_wheel_joint</joint_name>
+      <joint_name>right_wheel_joint</joint_name>
+    </plugin>
+  </gazebo>
 </robot>

File: description/urdf/robot_lidar.xacro (robot description, xacro)
@@ -1,62 +1,69 @@
 <?xml version="1.0"?>
-<robot xmlns:xacro="http://www.ros.org/wiki/xacro" >
-    <joint name="laser_joint" type="fixed">
-        <parent link="chassis_link"/>
-        <child link="laser_frame"/>
-        <origin xyz="${lidar_offset_X} 0 ${(chassis_height/2) + (lidar_stand_height) + (lidar_height/2)}" rpy="0 0 0"/>
-    </joint>
-    <link name="laser_frame">
-        <visual>
-            <geometry>
-                <cylinder radius="${lidar_radius}" length="${lidar_height}"/>
-            </geometry>
-            <material name="red"/>
-        </visual>
-        <collision>
-            <geometry>
-                <cylinder radius="${lidar_radius}" length="${lidar_height}"/>
-            </geometry>
-        </collision>
-        <xacro:inertial_cylinder mass="${lidar_mass}" length="${lidar_height}" radius="${lidar_radius}">
-            <origin xyz="0 0 0" rpy="0 0 0"/>
-        </xacro:inertial_cylinder>
-    </link>
-    <gazebo reference="laser_frame">
-        <material>Gazebo/Red</material>
-        <!--sensor name="laser" type="ray" JHP 2024.10.03-->
-	    <sensor name="laser_frame" type="gpu_lidar">
-            <pose> 0.0 0.0 0.0 0.0 0.0 0.0 </pose>
-            <visualize>true</visualize>
-            <update_rate>10</update_rate>
-            <topic>gz_scan</topic>
-            <gz_frame_id>laser_frame</gz_frame_id>
-            <frame_id>laser_frame</frame_id>
-            <ray>
-                <scan>
-                    <horizontal>
-                        <samples>360</samples>
-                        <resolution>1</resolution>
-                        <min_angle>-${pi}</min_angle>
-                        <max_angle>${pi}</max_angle>
-                    </horizontal>
-                    <vertical>
-                        <samples>1</samples>
-                        <resolution>1</resolution>
-                        <min_angle>0.0</min_angle>
-                        <max_angle>0.0</max_angle>
-                    </vertical>
-                </scan>
-                <range>
-                    <min>0.3</min>
-                    <max>12</max>
-                    <resolution>0.01</resolution>
-                </range>
-                <noise>
-                    <type>gaussian</type>
-                    <mean>0</mean>
-                    <stddev>0.01</stddev>
-                </noise>
-            </ray>
-        </sensor>
-    </gazebo>
+<robot xmlns:xacro="http://www.ros.org/wiki/xacro">
+  <joint name="laser_joint" type="fixed">
+    <parent link="chassis_link"/>
+    <child link="laser_frame"/>
+    <origin xyz="${lidar_offset_X} 0 ${(chassis_height/2) + (lidar_stand_height) + (lidar_height/2)}" rpy="0 0 0"/>
+  </joint>
+  <link name="laser_frame">
+    <visual>
+      <geometry>
+        <cylinder radius="${lidar_radius}" length="${lidar_height}"/>
+      </geometry>
+      <material name="red"/>
+    </visual>
+    <collision>
+      <geometry>
+        <cylinder radius="${lidar_radius}" length="${lidar_height}"/>
+      </geometry>
+    </collision>
+    <xacro:inertial_cylinder mass="${lidar_mass}" length="${lidar_height}" radius="${lidar_radius}">
+      <origin xyz="0 0 0" rpy="0 0 0"/>
+    </xacro:inertial_cylinder>
+  </link>
+  <gazebo reference="laser_frame">
+    <material>Gazebo/Red</material>
+    <!--sensor name="laser" type="ray" JHP 2024.10.03-->
+    <sensor name="laser_frame" type="gpu_lidar">
+      <pose> 0.0 0.0 0.0 0.0 0.0 0.0 </pose>
+      <visualize>true</visualize>
+      <update_rate>10</update_rate>
+      <topic>gz_scan</topic>
+      <gz_frame_id>laser_frame</gz_frame_id>
+      <frame_id>laser_frame</frame_id>
+      <lidar>
+        <scan>
+          <horizontal>
+            <samples>360</samples>
+            <resolution>1</resolution>
+            <min_angle>-${pi}</min_angle>
+            <max_angle>${pi}</max_angle>
+          </horizontal>
+          <vertical>
+            <samples>1</samples>
+            <resolution>1</resolution>
+            <min_angle>0.0</min_angle>
+            <max_angle>0.0</max_angle>
+          </vertical>
+        </scan>
+        <range>
+          <min>0.3</min>
+          <max>12</max>
+          <resolution>0.01</resolution>
+        </range>
+        <noise>
+          <type>gaussian</type>
+          <mean>0</mean>
+          <stddev>0.01</stddev>
+        </noise>
+      </lidar>
+    </sensor>
+    <!-- Add the gazebo_ros plugin -->
+    <plugin name="gazebo_ros_laser_controller" filename="libgazebo_ros_gpu_laser.so">
+      <alwaysOn>true</alwaysOn>
+      <updateRate>10</updateRate>
+      <topicName>/scan</topicName>
+      <frameName>laser_frame</frameName>
+    </plugin>
+  </gazebo>
 </robot>
